File: Osiris_PDB_RevA.kicad_sch (KiCad schematic)
At the start: 14 parts, among them J1 BATTERY_IN_4S, J2 ESC1_OUT, J3 ESC2_OUT, J4 ESC3_OUT, J5 ESC4_OUT, J6 OSIRIS_OUT_XT60_M_PIGTAIL

Commit message: FIX
FIX
Parts:
- removed C1: 1000uF 35V LOW-ESR, Capacitor_THT:CP_Radial_D12.5mm_P5.00mm, symbol Device:C_Polarized
- removed C5: 100uF 35V DNP, Capacitor_THT:CP_Radial_D8.0mm_P3.50mm, symbol Device:C_Polarized
- removed D1, D2: SMCJ17CA, Diode_SMD:D_SMC, symbol Device:D_TVS
- removed J2: ESC1_OUT, Connector_Wire:SolderWire-4sqmm_1x02_P12mm_D3mm_OD6mm, symbol Connector_Generic:Conn_01x02
- removed J3: ESC2_OUT, Connector_Wire:SolderWire-4sqmm_1x02_P12mm_D3mm_OD6mm, symbol Connector_Generic:Conn_01x02
- removed J4: ESC3_OUT, Connector_Wire:SolderWire-4sqmm_1x02_P12mm_D3mm_OD6mm, symbol Connector_Generic:Conn_01x02
- removed J5: ESC4_OUT, Connector_Wire:SolderWire-4sqmm_1x02_P12mm_D3mm_OD6mm, symbol Connector_Generic:Conn_01x02
- removed J6: OSIRIS_OUT_XT60_M_PIGTAIL, Connector_Wire:SolderWire-2sqmm_1x02_P7.8mm_D2mm_OD3.9mm, symbol Connector_Generic:Conn_01x02
- added C1: 5n6, symbol Device:C
- added C5: C, symbol Device:C
- added C6: 10u, symbol Device:C
- added Q1, Q2: ISC015N06NM5LF2, symbol PDB_Symbols:ISC015N06NM5LF2
- added R1: 2M0, symbol Device:R
- added R2: 43k2, symbol Device:R
- added R3: 56k2, symbol Device:R
- added R4: 22k, symbol Device:R
- added R5: FC4L64R005FER, PDB_Footprints:OH_FC4L64_OHM, symbol PDB_Symbols:FC4L64R005FER
- added R6: 680k, symbol Device:R
- added R7: 200k, symbol Device:R
- added R8, R9: R, symbol Device:R
- added U1: LTC4368IMS-1-PBF, MS_10_ADI, symbol PDB_Symbols:LTC4368IMS-1-PBF
- added U2: INA228AIDGSR, VSSOP10_DGS_TEX, symbol PDB_Symbols:INA228AIDGSR
- added U3: TPS7A1633DGNR, DGN0008C_N, symbol PDB_Symbols:TPS7A1633DGNR
- C2: value 100nF 50V X7R -> 1U0; footprint Capacitor_SMD:C_0805_2012Metric -> (none)
- C3: value 1uF 50V X7R -> 100n; footprint Capacitor_SMD:C_0805_2012Metric -> (none)
- C4: value 100nF 50V X7R -> 10u; footprint Capacitor_SMD:C_0805_2012Metric -> (none)
- F1: value 0678H6300-02 6.3A -> Fuse; footprint PDB_Footprints:FUSC9830X318N -> (none)
- J1: value BATTERY_IN_4S -> XT60; footprint Connector_Wire:SolderWire-4sqmm_1x02_P12mm_D3mm_OD6mm -> (none)
Connections:
- net GND: now also C4.1, J1.1 (Pin_1), C1.2, C5.2, C6.1, R3.2, R7.1, U1.5 (GND), U2.1 (A1), U2.2 (A0), U2.7 (GND), U3.4 (GND), U3.9 (PAD); no longer C4.2, J1.2 (Pin_2)
- removed net OSIRIS_FUSED: C3.1, C4.1, F1.2
- removed net VBAT: C2.1, F1.1, J1.1 (Pin_1)
- new net: C1.1, R4.2
- new net: R9.2, U2.10 (IN+)
- new net: R8.2, U2.9 (IN-)
- new net: R2.2, R3.1, U1.3 (OV)
- new net: R1.2, R2.1, U1.2 (UV)
- new net: C3.1, U1.4 (RETRY)
- new net GATE_DRV: Q1.4 (GATE), Q2.4 (GATE), R4.1, U1.10 (GATE)
- new net INA_ALERT: U2.3 (ALERT)
- new net INA_IN_N: R8.1
- new net INA_IN_P: R9.1
- new net PDB_3V3: C5.1, C6.2, U2.6 (VS), U3.1 (OUT)
- new net PDB_I2C_SCL: U2.5 (SCL)
- new net PDB_I2C_SDA: U2.4 (SDA)
- new net PDB_PROTECTED: Q2.5 (DRAIN), Q2.6 (DRAIN), Q2.7 (DRAIN), Q2.8 (DRAIN), R5.1
- new net PDB_VOUT: C4.2, R5.4, U2.8 (VBUS), U3.5 (EN), U3.8 (IN)
- new net SHDN_LTC: R6.1, R7.2, U1.6 (*SHDN)
- new net SHUNT_HI: R5.2, U1.9 (SENSE)
- new net SHUNT_LO: C2.1, R5.3, U1.8 (VOUT)
- new net SW_COMMON: Q1.1 (SOURCE), Q1.2 (SOURCE), Q1.3 (SOURCE), Q2.1 (SOURCE), Q2.2 (SOURCE), Q2.3 (SOURCE)
- new net VBAT_FUSED: F1.2, Q1.5 (DRAIN), Q1.6 (DRAIN), Q1.7 (DRAIN), Q1.8 (DRAIN), R1.1, R6.2, U1.1 (VIN)
- new net VBAT_RAW: F1.1, J1.2 (Pin_2)
- no-connect marks 0 -> 4
Other:
- note removed: "4S BATTERY AND FOUR EXTERNAL ESC BRANCHES"
- note removed: "C5 DNP until hot-plug testing establishes a need."
- note removed: "FUSED RAW-4S OSIRIS BRANCH"
- company: Osiris UAV -> (none)
- title: Osiris 4S Power Distribution Board -> (none)

Commit message: FIX
Parts:
- C5: value C -> 100n
- R8, R9: value R -> 10
Connections:
- net INA_IN_N: now also R8.2, U2.9 (IN-); no longer R8.1
- net INA_IN_P: now also R9.2, U2.10 (IN+); no longer R9.1
- net SHUNT_HI: now also R9.1
- net SHUNT_LO: now also R8.1
- net INA_ALERT renamed INA_ALERT_N
Other:
- moved on the sheet: R8, R9

Commit message: Consolidate Rev A schematic, component libraries and readiness review
Parts:
- added C7, C8: 100n, Capacitor_SMD:C_0603_1608Metric, symbol Device:C
- added C9: 10u, Capacitor_SMD:C_1206_3216Metric, symbol Device:C
- added D1: SMAJ24CA, Diode_SMD:D_SMA, symbol Device:D_TVS
- added D2, D3: MBR0540, Diode_SMD:D_SOD-123, symbol Device:D_Schottky
- added J2: OSIRIS_I2C, Connector_JST:JST_GH_BM04B-GHS-TBT_1x04-1MP_P1.25mm_Vertical, symbol Connector_Generic:Conn_01x04
- added J3: XT60PW-F, Connector_AMASS:AMASS_XT60PW-F_1x02_P7.20mm_Horizontal, symbol PDB_Symbols:XT60PW_F
- added R10: 4k7, Resistor_SMD:R_0805_2012Metric, symbol Device:R
- added TP1, TP2, TP3, TP4, TP5, TP6, TP7: TestPoint, TestPoint:TestPoint_Pad_D1.5mm, symbol Connector:TestPoint
- added U4: 74AUP1G07GW, Package_TO_SOT_SMD:SOT-353_SC-70-5, symbol 74xGxx:74AUP1G07
- C1: footprint (none) -> Capacitor_SMD:C_0805_2012Metric; MPN (none) -> C2012C0G2A562J125AA; Manufacturer (none) -> TDK; Selection_Status (none) -> CGATE at the U1 GATE pin per requirements D2; sets the 6.25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
- C2: footprint (none) -> Capacitor_SMD:C_0805_2012Metric; MPN (none) -> C2012X7R1H105K125AB; Manufacturer (none) -> TDK; Selection_Status (none) -> Nominal specification verified; DC-bias and circuit validat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
- C3, C5: footprint (none) -> Capacitor_SMD:C_0603_1608Metric; MPN (none) -> C0603C104K4RACTU; Manufacturer (none) -> KEMET; Selection_Status (none) -> Nominal specification verified; DC-bias and circuit validat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
- C4: footprint (none) -> Capacitor_SMD:C_1206_3216Metric; MPN (none) -> C3216X7R1H106K160AC; Manufacturer (none) -> TDK; Selection_Status (none) -> 10 uF local U3 input capacitor on protected PDB_VOUT.
- C6: footprint (none) -> Capacitor_SMD:C_0805_2012Metric; MPN (none) -> C2012X7R1A106K125AC; Manufacturer (none) -> TDK; Selection_Status (none) -> Nominal specification verified; DC-bias and circuit validat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
- F1: value Fuse -> 4A MINI; footprint (none) -> Fuse:Fuseholder_Blade_Mini_Keystone_3568; Holder_Datasheet (none) -> ${KIPRJMOD}/Datasheets/Keystone_3568.pdf; Holder_MPN (none) -> 3568; Holder_Manufacturer (none) -> Keystone Electronics; MPN (none) -> 0297004.WXNV; Manufacturer (none) -> Littelfuse; Selection_Status (none) -> PROVISIONAL 4 A candidate. 2.22 A is an assumed operating s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
- J1: value XT60 -> XT60PW-M; footprint (none) -> Connector_AMASS:AMASS_XT60PW-M_1x02_P7.20mm_Horizontal; MPN (none) -> XT60PW-M; Manufacturer (none) -> AMASS; Selection_Status (none) -> Assigned; verify cable mating, polarity and board-edge clea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
- Q1, Q2: footprint (none) -> PDB_Footprints:ISC015N06NM5LF2_TDSON8FL; MPN (none) -> ISC015N06NM5LF2; Manufacturer (none) -> Infineon
- R1, R2: footprint (none) -> Resistor_SMD:R_0805_2012Metric; Selection_Status (none) -> Package assigned; MPN and power/tolerance validation pending; Tolerance (none) -> 1%
- R3, R6, R7, R8, R9: footprint (none) -> Resistor_SMD:R_0805_2012Metric; Selection_Status (none) -> Package assigned; MPN and power/tolerance validation pending
- R4: footprint (none) -> Resistor_SMD:R_0805_2012Metric; Selection_Status (none) -> RGATE in the LTC4368 Figure 11 series position per requirem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; Tolerance (none) -> 1%
- R5: MPN (none) -> FC4L64R005FER; Manufacturer (none) -> Ohmite
- U1: footprint MS_10_ADI -> PDB_Footprints:MS_10-MSOP_ADI; MPN (none) -> LTC4368IMS-1#PBF; Manufacturer (none) -> Analog Devices
- U2: footprint VSSOP10_DGS_TEX -> PDB_Footprints:VSSOP10_DGS_TEX; MPN (none) -> INA228AIDGSR; Manufacturer (none) -> Texas Instruments
- U3: footprint DGN0008C_N -> PDB_Footprints:DGN0008C_N; MPN (none) -> TPS7A1633DGNR; Manufacturer (none) -> Texas Instruments; Selection_Status (none) -> Supplied from protected PDB_VOUT; loses power during a trip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
Connections:
- net GND: now also C8.1, C9.2, D1.2 (A2), D3.2 (A), J2.4 (Pin_4), J3.1 (-), TP3.1, U4.3 (GND)
- net INA_ALERT_N: now also TP6.1, U4.4; no longer U2.3 (ALERT)
- net INA_IN_N: now also C7.2
- net INA_IN_P: now also C7.1
- net PDB_3V3: now also C8.2, R10.1, TP5.1, U4.5 (VCC)
- net PDB_I2C_SCL: now also J2.2 (Pin_2)
- net PDB_I2C_SDA: now also J2.3 (Pin_3)
- net PDB_PROTECTED: now also TP2.1
- net PDB_VOUT: now also C9.1, D3.1 (K), J3.2 (+), TP4.1
- net VBAT_FUSED: now also D1.1 (A1), TP1.1
- net GATE_PIN: now reaches C1.1, R4.2
- net GATE_PIN: now also U1.10 (GATE), D2.1 (K)
- net PDB_FAULT_N: now reaches U1.7 (FAULT)
- net PDB_FAULT_N: now also TP7.1
- net GATE_DRV renamed GATE_FET
- net GATE_FET: now also D2.2 (A); no longer U1.10 (GATE)
- new net INA_ALERT_LOCAL_N: R10.2, U2.3 (ALERT), U4.2
- no-connect marks 4 -> 6
Other:
- note added: "J2 mates 1:1 with Osiris J28 (FMU_I2C1). Verify Osiris R74/R75 pull-up supply and rise time. Rev A: +3V3; imported PCB: ST_LINK_T_PWR. U2 address is 0x40; Osiris IC11 is 0x45 on the internal FMU_I2C4 bus, so there is no clash. Osiris Rev A exposes no spare GPIO or +3V3 on any GH connector, so INA_ALERT_N and PDB_FAULT_N go to TP6/TP7 only. Add pull-ups at whatever consumes them in a later revisio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"
- note added: "Planning case: 2.22 A at 10.56 V; load validation pending. F1: 4 A MINI provisional (0297004.WXNV) in a Keystone 3568 holder. 10 A nominal electronic breaker; fault coordination pending. Gate network per LTC4368 Figure 11: C1 at the GATE pin, R4 in series to the FETs, D2 across R4 for fast turn-off. D1 is bidirectional; a unidirectional TVS would short a reversed pack and defeat the reverse-batte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"
- moved on the sheet: C1, C2, C3, C4, C5, C6, F1, J1, Q1, Q2, R1, R2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

Commit message: Freeze A-P1 procurement baseline and feeder planning package
Parts:
- Q1, Q2: MPN ISC015N06NM5LF2 -> ISC015N06NM5LF2ATMA1; Selection_Status (none) -> Full Infineon tape-and-reel order code; same ISC015N06NM5LF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
- R1: MPN (none) -> RC0805FR-072ML; Manufacturer (none) -> YAGEO; Selection_Status Package assigned; MPN and power/tolerance validation pending -> Procurement baseline: nominal value and 0805 footprint reta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
- R10: MPN (none) -> RC0805FR-074K7L; Manufacturer (none) -> YAGEO; Selection_Status Package assigned; MPN and power/tolerance validation pending -> Procurement baseline: nominal value and 0805 footprint reta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
- R2: MPN (none) -> RC0805FR-0743K2L; Manufacturer (none) -> YAGEO; Selection_Status Package assigned; MPN and power/tolerance validation pending -> Procurement baseline: nominal value and 0805 footprint reta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
- R3: MPN (none) -> RC0805FR-0756K2L; Manufacturer (none) -> YAGEO; Selection_Status Package assigned; MPN and power/tolerance validation pending -> Procurement baseline: nominal value and 0805 footprint reta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
- R4: MPN (none) -> RC0805FR-0722KL; Manufacturer (none) -> YAGEO; Selection_Status RGATE in the LTC4368 Figure 11 series position per requirem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 -> Procurement baseline: nominal value and 0805 footprint reta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
- R6: MPN (none) -> RC0805FR-07680KL; Manufacturer (none) -> YAGEO; Selection_Status Package assigned; MPN and power/tolerance validation pending -> Procurement baseline: nominal value and 0805 footprint reta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
- R7: MPN (none) -> RC0805FR-07200KL; Manufacturer (none) -> YAGEO; Selection_Status Package assigned; MPN and power/tolerance validation pending -> Procurement baseline: nominal value and 0805 footprint reta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
- R8, R9: MPN (none) -> RC0805FR-0710RL; Manufacturer (none) -> YAGEO; Selection_Status Package assigned; MPN and power/tolerance validation pending -> Procurement baseline: nominal value and 0805 footprint reta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
- U1: MPN LTC4368IMS-1#PBF -> LTC4368IMS-1#TRPBF; Selection_Status (none) -> Tape-and-reel order code selected for assembly; same indust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
Other:
- note added: "Reference: old Osiris J28 (FMU_I2C1). New Rev B ports/power not drawn; verify interface. Verify Osiris R74/R75 pull-up supply and rise time. Rev A: +3V3; imported PCB: ST_LINK_T_PWR. U2 address is 0x40; Osiris IC11 is 0x45 on the internal FMU_I2C4 bus, so there is no clash. Osiris Rev A exposes no spare GPIO or +3V3 on any GH connector, so INA_ALERT_N and PDB_FAULT_N go to TP6/TP7 only. Add pull-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"
- note removed: "J2 mates 1:1 with Osiris J28 (FMU_I2C1). Verify Osiris R74/R75 pull-up supply and rise time. Rev A: +3V3; imported PCB: ST_LINK_T_PWR. U2 address is 0x40; Osiris IC11 is 0x45 on the internal FMU_I2C4 bus, so there is no clash. Osiris Rev A exposes no spare GPIO or +3V3 on any GH connector, so INA_ALERT_N and PDB_FAULT_N go to TP6/TP7 only. Add pull-ups at whatever consumes them in a later revisio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"
- title: (none) -> Osiris PDB - procurement baseline

Commit message: update 9/17/26
Parts:
- removed D2: MBR0540, Diode_SMD:D_SOD-123, symbol Device:D_Schottky
- added C10: 100n, Capacitor_SMD:C_0603_1608Metric, symbol Device:C
- added C11, C12, C13, C14, C15, C16: 1u, Capacitor_THT:C_Rect_L7.2mm_W4.5mm_P5.00mm, symbol Device:C
- added D4: SMAJ24CA, Diode_SMD:D_SMA, symbol Device:D_TVS
- added Q3: BSC070N10NS5, Package_TO_SOT_SMD:TDSON-8-1, symbol PDB_Symbols:BSC070N10NS5
- added R11: 1k58, Resistor_SMD:R_0805_2012Metric, symbol Device:R
- added R12: 1k0, Resistor_SMD:R_0805_2012Metric, symbol Device:R
- added R13: 54k9, Resistor_SMD:R_0805_2012Metric, symbol Device:R
- added R14: 22M, Resistor_SMD:R_0805_2012Metric, symbol Device:R
- added R15, R16: 10k, Resistor_SMD:R_0805_2012Metric, symbol Device:R
- added R17, R18: 4k7, Resistor_SMD:R_0805_2012Metric, symbol Device:R
- added R19: 1k, Resistor_SMD:R_2512_6332Metric, symbol Device:R
- added R20: 1, Resistor_SMD:R_2512_6332Metric, symbol Device:R
- added R21: 100, Resistor_SMD:R_0805_2012Metric, symbol Device:R
- added U5: LTC4359IMS8, Package_SO:MSOP-8_3x3mm_P0.65mm, symbol PDB_Symbols:LTC4359IMS8
- C1: value 5n6 -> 22n; MPN C2012C0G2A562J125AA -> C2012C0G2A223J125AC; Selection_Status CGATE at the U1 GATE pin per requirements D2; sets the 6.25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 -> 22 nF 5% C0G in series with R4 from GATE_PIN to GND. PDB-on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
- C6: Selection_Status Nominal specification verified; DC-bias and circuit validat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 -> A-P2 LT3010 output capacitor: require >=1 uF effective over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
- C9: Selection_Status Local bulk at the output connector; keeps total load capaci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 -> Output bulk capacitor; final total downstream capacitance a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
- D1: Selection_Status Bidirectional so reverse-battery blocking is preserved; bre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 -> Bidirectional 24 V TVS candidate; 38.9 V specified clamp is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
- D3: value MBR0540 -> STPST10H100SB; footprint Diode_SMD:D_SOD-123 -> PDB_Footprints:STPST10H100SB_DPAK; MPN MBR0540T1G -> STPST10H100SB-TR; Manufacturer onsemi -> STMicroelectronics; Selection_Status Output negative-voltage clamp; verify worst-case forward vo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 -> Selected power clamp. Connect both anode leads to GND and c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
- F1: Selection_Status PROVISIONAL 4 A candidate. 2.22 A is an assumed operating s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 -> 4 A 32 V MINI; load envelope 2.5 A maximum. Fuse, source an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
- J2: Selection_Status Re-pinned per requirements D3 to match Osiris J28 with a st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 -> PDB pinout fixed; Osiris R74/R75 12k pull-ups to switched 3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
- J3: Selection_Status Assigned with dedicated symbol pin mapping; verify physical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 -> PDB polarity fixed. Verify physical cable contacts and boar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
- Q1, Q2: Selection_Status Full Infineon tape-and-reel order code; same ISC015N06NM5LF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 -> (none)
- R1: value 2M0 -> 237k; MPN RC0805FR-072ML -> RC0805FR-07237KL; Selection_Status Procurement baseline: nominal value and 0805 footprint reta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 -> 1% 0805 UV divider. Selected for cold-start threshold margi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
- R10, R6, R7, R8, R9: Selection_Status Procurement baseline: nominal value and 0805 footprint reta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 -> Package assigned; MPN and power/tolerance validation pending
- R2: value 43k2 -> 11k8; MPN RC0805FR-0743K2L -> RC0805FR-0711K8L; Selection_Status Procurement baseline: nominal value and 0805 footprint reta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 -> 1% 0805; lower UV divider resistor.
- R3: value 56k2 -> 2M0; MPN RC0805FR-0756K2L -> RC0805FR-072ML; Selection_Status Procurement baseline: nominal value and 0805 footprint reta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 -> Package assigned; MPN and power/tolerance validation pending
- R4: Selection_Status Procurement baseline: nominal value and 0805 footprint reta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 -> U1 GATE directly drives Q1/Q2. R4 is in series with C1 to g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
- R5: value FC4L64R005FER -> 5m; Selection_Status (none) -> 5 mOhm 1% 2 W four-terminal. Nominal breaker 10 A; normal-c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
- U1: Selection_Status Tape-and-reel order code selected for assembly; same indust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 -> (none)
- U3: value TPS7A1633DGNR -> LT3010EMS8E; footprint PDB_Footprints:DGN0008C_N -> Package_SO:MSOP-8-1EP_3x3mm_P0.65mm_EP1.68x1.88mm; symbol PDB_Symbols:TPS7A1633DGNR -> PDB_Symbols:LT3010EMS8E; MPN TPS7A1633DGNR -> LT3010EMS8E#TRPBF; Manufacturer Texas Instruments -> Analog Devices; Selection_Status Supplied from protected PDB_VOUT; loses power during a trip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 -> A-P2 engineering draft: reverse-input/current-protected LT3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
Connections:
- net GATE_FET is gone; now on net GATE_PIN: Q1.4 (GATE), Q2.4 (GATE), R4.1
- net GATE_PIN: now also R14.1; no longer C1.1, R4.2
- net GND: now also R2.2, C12.2, C13.2, C14.2, C16.2, R12.2, R13.2, R19.2; no longer R3.2
- net INA_ALERT_N: now also R16.2
- net INA_IN_N: now also C13.1
- net INA_IN_P: now also C12.1
- net PDB_3V3: now also C10.1, R11.1, R15.1, R16.1, R17.1, R18.1
- net PDB_FAULT_N: now also R15.2
- net PDB_I2C_SCL: now also R17.2
- net PDB_I2C_SDA: now also R18.2
- net PDB_VOUT: now also R21.1; no longer U2.8 (VBUS)
- net VBAT_FUSED: now also R3.1, C11.1, C15.1, Q3.5 (DRAIN), Q3.6 (DRAIN), Q3.7 (DRAIN), Q3.8 (DRAIN), U5.8 (OUT); no longer F1.2, TP1.1
- net LTC_UV: now reaches R1.2, R2.1, U1.2 (UV)
- net LTC_UV: now also R14.2
- net PDB_LDO_ADJ: now reaches U3.2 (ADJ)
- net PDB_LDO_ADJ: now also C10.2, R11.2, R12.1
- new net GATE_RC: C1.1, R4.2
- new net IDEAL_GATE: Q3.4 (GATE), U5.1 (GATE)
- new net IDEAL_IN: D4.2 (A2), F1.2, Q3.1 (SOURCE), Q3.2 (SOURCE), Q3.3 (SOURCE), R20.1, TP1.1, U5.2 (SOURCE), U5.4 (IN), U5.5 (SHDN)
- new net IDEAL_VSS: C11.2, C15.2, D4.1 (A1), R19.1, U5.6 (VSS)
- new net INA_VBUS: C14.1, R21.2, U2.8 (VBUS)
- new net INPUT_DAMP: C16.1, R20.2
- new net LTC_OV: R13.1, R3.2, U1.3 (OV)
- no-connect marks 6 -> 7
Other:
- note added: "4S input: 12-16.8 V normal. Proposed load: <=25 W AND <=2.5 A. Startup capacitance: <=220 uF worst-case. GATE directly drives Q1/Q2. R4 + C1 form a series branch to GND. Existing Osiris input circuitry retained. Load model includes the planned 7 W Jetson mode. A-P4-DRAFT: PCB and bench validation required. U5/Q3 block reverse current; D3 clamps output. See Simulation/closure-20260915/RELEASE.md."
- note added: "C11-C16: 1 uF, 63 V, 5% film. C11 + C15 provide 2 uF. Place C12/C13 and R8/R9 symmetrically at U2. R21/C14: allow 1 ms settling before valid VBUS readings. Keep U5, Q3, D4 and C11/C15 loops short; R20/C16 at the input."
- note added: "J2: 1 NC, 2 SCL, 3 SDA, 4 GND. R17/R18 DNP; host supplies 3.3 V pull-ups. 100 kHz; <=90 pF total with Osiris 12k pull-ups. Verify unpowered behavior and cable pinout. INA228: address 0x40, ADCRANGE=0. R5=5 mOhm; 50 uA/LSB: SHUNT_CAL=3277. Calibrate assembled board. FAULT / ALERT: TP7 / TP6 only."
- note added: "LOW-LOSS REVERSE INPUT PROTECTION"
- note added: "SENSOR INPUT FILTERS"
- note removed: "Planning case: 2.22 A at 10.56 V; load validation pending. F1: 4 A MINI provisional (0297004.WXNV) in a Keystone 3568 holder. 10 A nominal electronic breaker; fault coordination pending. Gate network per LTC4368 Figure 11: C1 at the GATE pin, R4 in series to the FETs, D2 across R4 for fast turn-off. D1 is bidirectional; a unidirectional TVS would short a reversed pack and defeat the reverse-batte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"
- note removed: "Reference: old Osiris J28 (FMU_I2C1). New Rev B ports/power not drawn; verify interface. Verify Osiris R74/R75 pull-up supply and rise time. Rev A: +3V3; imported PCB: ST_LINK_T_PWR. U2 address is 0x40; Osiris IC11 is 0x45 on the internal FMU_I2C4 bus, so there is no clash. Osiris Rev A exposes no spare GPIO or +3V3 on any GH connector, so INA_ALERT_N and PDB_FAULT_N go to TP6/TP7 only. Add pull-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"
- title: Osiris PDB - procurement baseline -> Osiris PDB - engineering draft
- moved on the sheet: D1, R3, R5
