File: Osiris_PDB_RevA.kicad_sch (KiCad schematic)
At the start: 59 parts, among them J1 XT60PW-M, J2 OSIRIS_I2C, J3 XT60PW-F, Q1 ISC015N06NM5LF2, Q2 ISC015N06NM5LF2, Q3 BSC070N10NS5, U1 LTC4368IMS-1-PBF, U2 INA228AIDGSR, U3 LT3010EMS8E, U4 74AUP1G07GW, U5 LTC4359IMS8

Commit message: 9/21/2026
Parts:
- U1: value LTC4368IMS-1-PBF -> LTC4368HMS-1-PBF; MPN LTC4368IMS-1#TRPBF -> LTC4368HMS-1#TRPBF
Changed lines of the file:
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@@
 			)
 		)
-		(property "Value" "LTC4368IMS-1-PBF"
+		(property "Value" "LTC4368HMS-1-PBF"
 			(at 198.1200 69.8500 0)
 			(show_name no)
@@
 			)
 		)
-		(property "Description" ""
+		(property "Description" "Approved H-temperature-grade LTC4368-1; pin/function-compatible with LTC4368IMS-1 and rated -40 C to 125 C"
 			(at 198.1200 69.8500 0)
 			(hide yes)
@@
 			)
 		)
-		(property "MPN" "LTC4368IMS-1#TRPBF"
+		(property "MPN" "LTC4368HMS-1#TRPBF"
 			(at 175.2600 81.2800 0)
 			(hide yes)

Commit message: Save current PDB schematic and layout updates
Parts:
- added H1, H2, H3, H4: MountingHole, MountingHole:MountingHole_3.2mm_M3_ISO14580, symbol Mechanical:MountingHole
- added J4: XT60PW-F, Connector_AMASS:AMASS_XT60PW-F_1x02_P7.20mm_Horizontal, symbol PDB_Symbols:XT60PW_F
Connections:
- net GND: now also J4.1 (-)
- net PDB_VOUT: now also J4.2 (+)
Other:
- moved on the sheet: C15, R19, R3

Commit message: Resolve PDB CAD checks and prepare assembly handoff drafts
Parts:
- D3: symbol Device:D_Schottky -> PDB_Symbols:D_Schottky_PDB
- J2: symbol Connector_Generic:Conn_01x04 -> PDB_Symbols:Conn_01x04_PDB
- Q3: footprint Package_TO_SOT_SMD:TDSON-8-1 -> PDB_Footprints:BSC070N10NS5_TDSON8
- U4: symbol 74xGxx:74AUP1G07 -> PDB_Symbols:74AUP1G07_PDB
Changed lines of the file:
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@@
 			)
 		)
-		(property "Footprint" "Package_TO_SOT_SMD:TDSON-8-1"
+		(property "Footprint" "PDB_Footprints:BSC070N10NS5_TDSON8"
 			(at 86.36 12.7 0)
 			(hide yes)
@@
 	)
 	(symbol
-		(lib_id "74xGxx:74AUP1G07")
+		(lib_id "PDB_Symbols:74AUP1G07_PDB")
 		(at 172.72 210.82 0)
 		(unit 1)
@@
 	)
 	(symbol
-		(lib_id "Connector_Generic:Conn_01x04")
+		(lib_id "PDB_Symbols:Conn_01x04_PDB")
 		(at 388.62 236.22 0)
 		(unit 1)
@@
 			)
 		)
-		(property "Description" "5 A, 32 VDC MINI blade fuse; backup protection for a fault the MOSFETs cannot interrupt"
+		(property "Description" "4 A, 32 VDC MINI blade fuse; backup protection for a fault the MOSFETs cannot interrupt"
 			(at 40.64 33.02 90)
 			(hide yes)
@@
 	)
 	(symbol
-		(lib_id "Device:D_Schottky")
+		(lib_id "PDB_Symbols:D_Schottky_PDB")
 		(at 345.44 55.88 270)
 		(unit 1)

Commit message: added power path for esc on schematic
Parts:
- added C17: 470u/35V, Capacitor_SMD:CP_Elec_10x10.5, symbol Device:C
- added C18: 1u/50V, Capacitor_SMD:C_0805_2012Metric, symbol Device:C
- added C19: 100n/50V, Capacitor_SMD:C_0805_2012Metric, symbol Device:C
- added D5: SMBJ24CA, Diode_SMD:D_SMB, symbol Device:D_TVS
- added F2: UHS 100A, symbol Device:Fuse
- J1: value XT60PW-M -> 125A TERM; footprint Connector_AMASS:AMASS_XT60PW-M_1x02_P7.20mm_Horizontal -> (none); MPN XT60PW-M -> 1932588; Manufacturer AMASS -> Phoenix Contact; Selection_Status Assigned; verify cable mating, polarity and board-edge clea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 -> PROVISIONAL: input must carry ESC plus avionics current. Fi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
- J3: renamed from J4; value XT60PW-F -> 125A TERM; footprint Connector_AMASS:AMASS_XT60PW-F_1x02_P7.20mm_Horizontal -> (none); MPN XT60PW-F -> 1932588; Manufacturer AMASS -> Phoenix Contact; Selection_Status PDB polarity fixed. Verify physical cable contacts and boar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 -> PROVISIONAL: size for 60 A continuous and 100 A for 30 s. F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
- J4: renamed from J3; Selection_Status PDB polarity fixed. Verify physical cable contacts and boar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 -> OSIRIS POWER ONLY. Verify physical cable contacts and board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
Connections:
- net GND: now also C17.2, C18.2, C19.2, D5.2 (A2)
- net PDB_VOUT: no longer J3.2 (+)
- net VBAT_RAW: now also F2.1
- new net ESC_VBAT: C17.1, C18.1, C19.1, D5.1 (A1), F2.2, J3.2 (+)
Other:
- note added: "A-P5 DRAFT: dedicated ESC branch added; PCB placement/routing is not updated. Avionics: J4 power + J2 I2C to Osiris. ESC: J3 only, directly from VBAT_RAW through F2. C11-C16: 1 uF / 63 V non-polar film. Keep local bypass capacitors close to their ICs."
- note added: "AVIONICS POWER | 4S BATTERY -> PROTECTED RAW 4S TO OSIRIS (JETSON 15 W MODE)"
- note added: "DEDICATED ESC POWER | 4S / 60 A CONTINUOUS / 100 A FOR 30 s (PROVISIONAL)"
- note added: "J3 ESC ONLY. F2/D5/C17-C19 bypass avionics F1, Q3, Q1/Q2, U1 and R5. Route ESC positive and return directly to the battery-entry star with matched high-current copper. Connector, fuse, heavy-copper land pattern, pack fault current, inrush and thermal rise require qualification."
- note removed: "MAIN POWER PATH | BATTERY -> PROTECTED RAW 4S TO OSIRIS"
- note removed: "Same electrical circuit; drawing rearranged only. No capacitor values or footprints changed. PDB supplies raw battery voltage; Osiris Rev B requires its replacement power section. C11-C16: 1 uF / 63 V non-polar film. Keep local bypass capacitors close to their ICs."
- moved on the sheet: J3

Commit message: esc
Connections:
- net ESC_VBAT is gone; now on net GND: C17.1, C18.1, C19.1, D5.1 (A1), F2.2, J3.2 (+)
- net GND: no longer J3.1 (-)

Commit message: Route compact three-XT60 PDB candidate
Parts:
- F2: footprint (none) -> PDB_Footprints:SCHURTER_UHS_8.4x9.4mm_PROVISIONAL
- J1: value 125A TERM -> XT60PW-M; footprint (none) -> Connector_AMASS:AMASS_XT60PW-M_1x02_P7.20mm_Horizontal; MPN 1932588 -> XT60PW-M30; Manufacturer Phoenix Contact -> AMASS; Selection_Status PROVISIONAL: input must carry ESC plus avionics current. Fi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 -> NOT CURRENT-QUALIFIED: XT60PW-M30 is rated 35 A; input must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
- J3: value 125A TERM -> XT60PW-F; footprint (none) -> Connector_AMASS:AMASS_XT60PW-F_1x02_P7.20mm_Horizontal; MPN 1932588 -> XT60PW-F30; Manufacturer Phoenix Contact -> AMASS; Selection_Status PROVISIONAL: size for 60 A continuous and 100 A for 30 s. F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 -> NOT CURRENT-QUALIFIED: XT60PW-F30 is rated 35 A; ESC target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
Connections:
- net GND: now also J3.1 (-); no longer C17.1, C18.1, C19.1, D5.1 (A1), F2.2, J3.2 (+)
- new net ESC_VBAT: C17.1, C18.1, C19.1, D5.1 (A1), F2.2, J3.2 (+)
Other:
- note added: "A-P5 DRAFT: compact three-XT60 PCB candidate routed; 60 A/100 A target remains unqualified. Avionics: J4 power + J2 I2C to Osiris. ESC: J3 only, directly from VBAT_RAW through F2. C11-C16: 1 uF / 63 V non-polar film. Keep local bypass capacitors close to their ICs."
- note added: "J3 ESC ONLY. F2/D5/C17-C19 bypass avionics F1, Q3, Q1/Q2, U1 and R5. Compact PCB candidate routes ESC positive on F.Cu and shared return on B.Cu. XT60 current rating, fuse land pattern, copper, pack fault current, inrush and thermal rise require qualification."
- note removed: "A-P5 DRAFT: dedicated ESC branch added; PCB placement/routing is not updated. Avionics: J4 power + J2 I2C to Osiris. ESC: J3 only, directly from VBAT_RAW through F2. C11-C16: 1 uF / 63 V non-polar film. Keep local bypass capacitors close to their ICs."
- note removed: "J3 ESC ONLY. F2/D5/C17-C19 bypass avionics F1, Q3, Q1/Q2, U1 and R5. Route ESC positive and return directly to the battery-entry star with matched high-current copper. Connector, fuse, heavy-copper land pattern, pack fault current, inrush and thermal rise require qualification."
Changed lines of the file:
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@@
 		)
 	)
-	(text "J3 ESC ONLY. F2/D5/C17-C19 bypass avionics F1, Q3, Q1/Q2, U1 and R5.\nRoute ESC positive and return directly to the battery-entry star with matched high-current copper.\nConnector, fuse, heavy-copper land pattern, pack fault current, inrush and thermal rise require qualification."
+	(text "J3 ESC ONLY. F2/D5/C17-C19 bypass avionics F1, Q3, Q1/Q2, U1 and R5.\nCompact PCB candidate routes ESC positive on F.Cu and shared return on B.Cu.\nXT60 current rating, fuse land pattern, copper, pack fault current, inrush and thermal rise require qualification."
 		(exclude_from_sim no)
 		(at 255.27 97.79 0)
@@
 		)
 	)
-	(text "A-P5 DRAFT: dedicated ESC branch added; PCB placement/routing is not updated.\nAvionics: J4 power + J2 I2C to Osiris. ESC: J3 only, directly from VBAT_RAW through F2.\nC11-C16: 1 uF / 63 V non-polar film. Keep local bypass capacitors close to their ICs."
+	(text "A-P5 DRAFT: compact three-XT60 PCB candidate routed; 60 A/100 A target remains unqualified.\nAvionics: J4 power + J2 I2C to Osiris. ESC: J3 only, directly from VBAT_RAW through F2.\nC11-C16: 1 uF / 63 V non-polar film. Keep local bypass capacitors close to their ICs."
 		(exclude_from_sim no)
 		(at 20.32 276.86 0)
@@
 	(wire
 		(pts
-			(xy 383.54 74.93) (xy 383.54 87.63)
+			(xy 378.46 72.39) (xy 383.54 72.39)
 		)
 		(stroke
@@
 		)
 	)
+	(label "GND"
+		(at 378.46 72.39 0)
+		(effects
+			(font
+				(size 1.016 1.016)
+			)
+			(justify left bottom)
+		)
+	)
 	(label "SHUNT_HI"
 		(at 336.55 175.26 0)
@@
 			)
 		)
-		(property "Footprint" ""
+		(property "Footprint" "PDB_Footprints:SCHURTER_UHS_8.4x9.4mm_PROVISIONAL"
 			(at 274.32 74.168 90)
 			(hide yes)
@@
 			)
 		)
-		(property "Value" "125A TERM"
+		(property "Value" "XT60PW-M"
 			(at 17.78 35.56 0)
 			(show_name no)
@@
 			)
 		)
-		(property "Footprint" ""
+		(property "Footprint" "Connector_AMASS:AMASS_XT60PW-M_1x02_P7.20mm_Horizontal"
 			(at 17.78 40.64 0)
 			(hide yes)
@@
 			)
 		)
-		(property "Datasheet" "https://www.phoenixcontact.com/en-de/products/pcb-terminal-block-mkdsp-25-2-1500-1932588"
+		(property "Datasheet" "${KIPRJMOD}/Datasheets/AMASS_XT60PW-M.pdf"
 			(at 17.78 40.64 0)
 			(hide yes)
@@
 			)
 		)
-		(property "Description" "High-current 4S battery input; pin 1 GND, pin 2 VBAT_RAW. Candidate terminal is Phoenix 1932588, 125 A nominal with specified conductor."
+		(property "Description" "4S battery input; pin 1 GND, pin 2 VBAT_RAW. XT60PW-M footprint study only; connector current rating does not meet the 60 A ESC plus avionics target."
 			(at 17.78 35.56 0)
 			(hide yes)
@@
 			)
 		)
-		(property "Selection_Status" "PROVISIONAL: input must carry ESC plus avionics current. Final footprint, wire gauge, torque, assembly method, polarity and thermal rise require qualification."
+		(property "Selection_Status" "NOT CURRENT-QUALIFIED: XT60PW-M30 is rated 35 A; input must carry ESC plus avionics current and a 100 A burst target. Do not fabricate until connector architecture is changed or qualified."
 			(at 17.78 40.64 0)
 			(hide yes)
@@
 			)
 		)
-		(property "Manufacturer" "Phoenix Contact"
+		(property "Manufacturer" "AMASS"
 			(at 17.78 40.64 0)
 			(hide yes)
@@
 			)
 		)
-		(property "MPN" "1932588"
+		(property "MPN" "XT60PW-M30"
 			(at 17.78 40.64 0)
 			(hide yes)
@@
 			)
 		)
-		(property "Value" "125A TERM"
+		(property "Value" "XT60PW-F"
 			(at 388.62 67.31 0)
 			(show_name no)
@@
 			)
 		)
-		(property "Footprint" ""
+		(property "Footprint" "Connector_AMASS:AMASS_XT60PW-F_1x02_P7.20mm_Horizontal"
 			(at 388.62 50.8 0)
 			(hide yes)
@@
 			)
 		)
-		(property "Datasheet" "https://www.phoenixcontact.com/en-de/products/pcb-terminal-block-mkdsp-25-2-1500-1932588"
+		(property "Datasheet" "${KIPRJMOD}/Datasheets/AMASS_XT60PW-F.pdf"
 			(at 388.62 50.8 0)
 			(hide yes)
@@
 			)
 		)
-		(property "Description" "Dedicated four-motor ESC output; pin 1 is the high-current battery return and pin 2 is ESC_VBAT after F2. Candidate terminal is Phoenix 1932588, 125 A nominal with specified conductor."
+		(property "Description" "Dedicated ESC output; pin 1 GND, pin 2 ESC_VBAT after F2. XT60PW-F footprint study only; connector current rating does not meet the 60 A/100 A target."
 			(at 388.62 45.72 0)
 			(hide yes)
@@
 			)
 		)
-		(property "Selection_Status" "PROVISIONAL: size for 60 A continuous and 100 A for 30 s. Final footprint, cable, assembly method, temperature rise, and mate must be qualified before release."
+		(property "Selection_Status" "NOT CURRENT-QUALIFIED: XT60PW-F30 is rated 35 A; ESC target is 60 A continuous and 100 A for 30 seconds. Do not fabricate until connector architecture is changed or qualified."
 			(at 388.62 50.8 0)
 			(hide yes)
@@
 			)
 		)
-		(property "Manufacturer" "Phoenix Contact"
+		(property "Manufacturer" "AMASS"
 			(at 388.62 50.8 0)
 			(hide yes)
@@
 			)
 		)
-		(property "MPN" "1932588"
+		(property "MPN" "XT60PW-F30"
 			(at 388.62 50.8 0)
 			(hide yes)

Commit message: Restore compact PDB layout shown in reference image
Parts:
- C17: value 470u/35V -> 470u 35V LOW-ESR
- C18: value 1u/50V -> 1u 50V X7R
- C19: value 100n/50V -> 100n 50V X7R
- F2: value UHS 100A -> SCHURTER UHS 100A 3-140-177 PROVISIONAL
- J1: value XT60PW-M -> MKDSP 25/2-15.00 PROVISIONAL; footprint Connector_AMASS:AMASS_XT60PW-M_1x02_P7.20mm_Horizontal -> PDB_Footprints:MKDSP25_2_15mm_PROVISIONAL; MPN XT60PW-M30 -> 1932588; Manufacturer AMASS -> Phoenix Contact; Selection_Status NOT CURRENT-QUALIFIED: XT60PW-M30 is rated 35 A; input must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 -> LAB DESIGN IN PROGRESS: verify exact terminal, footprint, c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
- J3: value XT60PW-F -> MKDSP 25/2-15.00 PROVISIONAL; footprint Connector_AMASS:AMASS_XT60PW-F_1x02_P7.20mm_Horizontal -> PDB_Footprints:MKDSP25_2_15mm_PROVISIONAL; symbol PDB_Symbols:XT60PW_F -> Connector_Generic:Conn_01x02; MPN XT60PW-F30 -> 1932588; Manufacturer AMASS -> Phoenix Contact; Selection_Status NOT CURRENT-QUALIFIED: XT60PW-F30 is rated 35 A; ESC target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 -> LAB DESIGN IN PROGRESS: verify exact terminal, footprint, c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
- J4: Selection_Status OSIRIS POWER ONLY. Verify physical cable contacts and board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 -> PDB polarity fixed. Verify physical cable contacts and boar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
Other:
- note added: "AVIONICS POWER | 4S BATTERY -> PROTECTED RAW 4S TO OSIRIS (25 W DESIGN CASE)"
- note added: "J3 ESC OUTPUT ONLY. F2/D5/C17-C19 bypass the separate J4 avionics branch. Phoenix lab PCB routes ESC positive on F.Cu and return through ground copper. J1 pack interface, fuse land pattern, copper, fault current and heating need verification."
- note added: "PHOENIX LAB PCB: J1 input, J3 ESC output after F2, J4 Osiris avionics output after F1. Planning load: 50 A ESC + 5 A J1 avionics allowance; design targets 60 A ESC continuous / 100 A for 30 s. These currents are not yet qualified by the saved copper, terminals, fuse or pack connector."
- note removed: "A-P5 DRAFT: compact three-XT60 PCB candidate routed; 60 A/100 A target remains unqualified. Avionics: J4 power + J2 I2C to Osiris. ESC: J3 only, directly from VBAT_RAW through F2. C11-C16: 1 uF / 63 V non-polar film. Keep local bypass capacitors close to their ICs."
- note removed: "AVIONICS POWER | 4S BATTERY -> PROTECTED RAW 4S TO OSIRIS (JETSON 15 W MODE)"
- note removed: "J3 ESC ONLY. F2/D5/C17-C19 bypass avionics F1, Q3, Q1/Q2, U1 and R5. Compact PCB candidate routes ESC positive on F.Cu and shared return on B.Cu. XT60 current rating, fuse land pattern, copper, pack fault current, inrush and thermal rise require qualification."
- title: Osiris PDB - engineering draft -> Osiris PDB - Phoenix lab board
Changed lines of the file:
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@@
 	(paper "A3")
 	(title_block
-		(title "Osiris PDB - engineering draft")
+		(title "Osiris PDB - Phoenix lab board")
 		(date "2026-09-29")
-		(rev "A-P5-DRAFT")
-		(comment 1 "Dedicated ESC branch draft; Osiris avionics remains separately protected")
+		(rev "PHOENIX-LAB-DRAFT")
+		(comment 1 "J1 common input; J3 ESC output; J4 protected Osiris avionics output")
 		(comment 2 "Electrical design draft - PCB and bench validation required")
 	)
@@
 		)
 	)
-	(text "J3 ESC ONLY. F2/D5/C17-C19 bypass avionics F1, Q3, Q1/Q2, U1 and R5.\nCompact PCB candidate routes ESC positive on F.Cu and shared return on B.Cu.\nXT60 current rating, fuse land pattern, copper, pack fault current, inrush and thermal rise require qualification."
+	(text "J3 ESC OUTPUT ONLY. F2/D5/C17-C19 bypass the separate J4 avionics branch.\nPhoenix lab PCB routes ESC positive on F.Cu and return through ground copper.\nJ1 pack interface, fuse land pattern, copper, fault current and heating need verification."
 		(exclude_from_sim no)
 		(at 255.27 97.79 0)
@@
 		)
 	)
-	(text "AVIONICS POWER  |  4S BATTERY -> PROTECTED RAW 4S TO OSIRIS (JETSON 15 W MODE)"
+	(text "AVIONICS POWER  |  4S BATTERY -> PROTECTED RAW 4S TO OSIRIS (25 W DESIGN CASE)"
 		(exclude_from_sim no)
 		(at 20.32 17.78 0)
@@
 		)
 	)
-	(text "A-P5 DRAFT: compact three-XT60 PCB candidate routed; 60 A/100 A target remains unqualified.\nAvionics: J4 power + J2 I2C to Osiris. ESC: J3 only, directly from VBAT_RAW through F2.\nC11-C16: 1 uF / 63 V non-polar film. Keep local bypass capacitors close to their ICs."
+	(text "PHOENIX LAB PCB: J1 input, J3 ESC output after F2, J4 Osiris avionics output after F1.\nPlanning load: 50 A ESC + 5 A J1 avionics allowance; design targets 60 A ESC continuous / 100 A for 30 s.\nThese currents are not yet qualified by the saved copper, terminals, fuse or pack connector."
 		(exclude_from_sim no)
 		(at 20.32 276.86 0)
@@
 			)
 		)
-		(property "Value" "UHS 100A"
+		(property "Value" "SCHURTER UHS 100A 3-140-177 PROVISIONAL"
 			(at 274.32 67.31 90)
 			(show_name no)
@@
 			)
 		)
-		(property "Value" "1u/50V"
+		(property "Value" "1u 50V X7R"
 			(at 349.25 80.01 0)
 			(show_name no)
@@
 			)
 		)
-		(property "Value" "470u/35V"
+		(property "Value" "470u 35V LOW-ESR"
 			(at 326.39 80.01 0)
 			(show_name no)
@@
 			)
 		)
-		(property "Selection_Status" "OSIRIS POWER ONLY. Verify physical cable contacts and board-edge clearance; do not connect the four-motor ESC here."
+		(property "Selection_Status" "PDB polarity fixed. Verify physical cable contacts and board-edge clearance; old Osiris J16 numbering is not the new Rev B interface."
 			(at 388.62 35.56 0)
 			(hide yes)
@@
 			)
 		)
-		(property "Value" "XT60PW-M"
+		(property "Value" "MKDSP 25/2-15.00 PROVISIONAL"
 			(at 17.78 35.56 0)
 			(show_name no)
@@
 			)
 		)
-		(property "Footprint" "Connector_AMASS:AMASS_XT60PW-M_1x02_P7.20mm_Horizontal"
+		(property "Footprint" "PDB_Footprints:MKDSP25_2_15mm_PROVISIONAL"
 			(at 17.78 40.64 0)
 			(hide yes)
@@
 			)
 		)
-		(property "Datasheet" "${KIPRJMOD}/Datasheets/AMASS_XT60PW-M.pdf"
+		(property "Datasheet" "https://www.phoenixcontact.com/en-ca/products/printed-circuit-board-terminal-mkdsp-25-2-1500-1932588"
 			(at 17.78 40.64 0)
 			(hide yes)
@@
 			)
 		)
-		(property "Description" "4S battery input; pin 1 GND, pin 2 VBAT_RAW. XT60PW-M footprint study only; connector current rating does not meet the 60 A ESC plus avionics target."
+		(property "Description" "4S battery input; pin 1 GND, pin 2 VBAT_RAW. Phoenix Contact 1932588 terminal; footprint and assembly require verification."
 			(at 17.78 35.56 0)
 			(hide yes)
@@
 			)
 		)
-		(property "Selection_Status" "NOT CURRENT-QUALIFIED: XT60PW-M30 is rated 35 A; input must carry ESC plus avionics current and a 100 A burst target. Do not fabricate until connector architecture is changed or qualified."
+		(property "Selection_Status" "LAB DESIGN IN PROGRESS: verify exact terminal, footprint, conductor, wave-solder process, and power-path temperature before full-current use."
 			(at 17.78 40.64 0)
 			(hide yes)
@@
 			)
 		)
-		(property "Manufacturer" "AMASS"
+		(property "Manufacturer" "Phoenix Contact"
 			(at 17.78 40.64 0)
 			(hide yes)
@@
 			)
 		)
-		(property "MPN" "XT60PW-M30"
+		(property "MPN" "1932588"
 			(at 17.78 40.64 0)
 			(hide yes)
@@
 			)
 		)
-		(property "Value" "100n/50V"
+		(property "Value" "100n 50V X7R"
 			(at 367.03 80.01 0)
 			(show_name no)
@@
 	)
 	(symbol
-		(lib_id "PDB_Symbols:XT60PW_F")
+		(lib_id "Connector_Generic:Conn_01x02")
 		(at 388.62 72.39 0)
 		(unit 1)
@@
 			)
 		)
-		(property "Value" "XT60PW-F"
+		(property "Value" "MKDSP 25/2-15.00 PROVISIONAL"
 			(at 388.62 67.31 0)
 			(show_name no)
@@
 			)
 		)
-		(property "Footprint" "Connector_AMASS:AMASS_XT60PW-F_1x02_P7.20mm_Horizontal"
+		(property "Footprint" "PDB_Footprints:MKDSP25_2_15mm_PROVISIONAL"
 			(at 388.62 50.8 0)
 			(hide yes)
@@
 			)
 		)
-		(property "Datasheet" "${KIPRJMOD}/Datasheets/AMASS_XT60PW-F.pdf"
+		(property "Datasheet" "https://www.phoenixcontact.com/en-ca/products/printed-circuit-board-terminal-mkdsp-25-2-1500-1932588"
 			(at 388.62 50.8 0)
 			(hide yes)
@@
 			)
 		)
-		(property "Description" "Dedicated ESC output; pin 1 GND, pin 2 ESC_VBAT after F2. XT60PW-F footprint study only; connector current rating does not meet the 60 A/100 A target."
+		(property "Description" "Dedicated ESC output after F2; pin 1 GND, pin 2 ESC_VBAT. Phoenix Contact 1932588 terminal; footprint and assembly require verification."
 			(at 388.62 45.72 0)
 			(hide yes)
@@
 			)
 		)
-		(property "Selection_Status" "NOT CURRENT-QUALIFIED: XT60PW-F30 is rated 35 A; ESC target is 60 A continuous and 100 A for 30 seconds. Do not fabricate until connector architecture is changed or qualified."
+		(property "Selection_Status" "LAB DESIGN IN PROGRESS: verify exact terminal, footprint, conductor, wave-solder process, and power-path temperature before full-current use."
 			(at 388.62 50.8 0)
 			(hide yes)
@@
 			)
 		)
-		(property "Manufacturer" "AMASS"
+		(property "Manufacturer" "Phoenix Contact"
 			(at 388.62 50.8 0)
 			(hide yes)
@@
 			)
 		)
-		(property "MPN" "XT60PW-F30"
+		(property "MPN" "1932588"
 			(at 388.62 50.8 0)
 			(hide yes)
