File: Osiris_PDB_RevA.kicad_sch (KiCad schematic)
At the start: 69 parts, among them J1 MKDSP 25/2-15.00 PROVISIONAL, J2 OSIRIS_I2C, J3 MKDSP 25/2-15.00 PROVISIONAL, J4 XT60PW-F, Q1 ISC015N06NM5LF2, Q2 ISC015N06NM5LF2, Q3 BSC070N10NS5, U1 LTC4368HMS-1-PBF, U2 INA228AIDGSR, U3 LT3010EMS8E, U4 74AUP1G07GW, U5 LTC4359IMS8

Commit message: Update PDB design and purchasing deliverables
Parts:
- C17: value 470u 35V LOW-ESR -> 470u 35V HYBRID; footprint Capacitor_SMD:CP_Elec_10x10.5 -> PDB_Footprints:CP_Elec_Panasonic_G16_10x16.5; symbol Device:C -> PDB_Symbols:CP_Elec_Panasonic; MPN (none) -> EEHZS1V471P; Manufacturer (none) -> Panasonic; Selection_Status PROVISIONAL 4S value; use 35 V minimum rating and qualify r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 -> Selected EEHZS1V471P G16; 10 mm diameter, 16.5 mm height. A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
- D5: Selection_Status PROVISIONAL: local transient suppressor only; not a substit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 -> SMBJ24CA retained for local ringing control. Clamp is not a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
- F2: value SCHURTER UHS 100A 3-140-177 PROVISIONAL -> UHS 100A 50V; footprint PDB_Footprints:SCHURTER_UHS_8.4x9.4mm_PROVISIONAL -> PDB_Footprints:Fuse_SCHURTER_UHS_8.4x9.4mm; Selection_Status PROVISIONAL: verify 60 A continuous temperature rise, 100 A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 -> Selected prototype fuse. Manufacturer pad pattern 3.4 x 6.1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
- J1, J3: value MKDSP 25/2-15.00 PROVISIONAL -> MKDSP 25/2-15.00; footprint PDB_Footprints:MKDSP25_2_15mm_PROVISIONAL -> PDB_Footprints:Connector_MKDSP25_2_15mm; symbol Connector_Generic:Conn_01x02 -> PDB_Symbols:Conn_01x02_Phoenix; Selection_Status LAB DESIGN IN PROGRESS: verify exact terminal, footprint, c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 -> Drawing checked 2026-10-01: 15 mm pole pitch, 3.8 mm paired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
Changed lines of the file:
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@@
 	(title_block
 		(title "Osiris PDB - Phoenix lab board")
-		(date "2026-09-29")
-		(rev "PHOENIX-LAB-DRAFT")
+		(date "2026-10-01")
+		(rev "A-P6-PROTOTYPE")
 		(comment 1 "J1 common input; J3 ESC output; J4 protected Osiris avionics output")
-		(comment 2 "Electrical design draft - PCB and bench validation required")
+		(comment 2 "4-layer 2 oz prototype - physical qualification pending")
 	)
 	(text "STATUS / OPTIONAL PULL-UPS"
@@
 			)
 		)
-		(property "Value" "SCHURTER UHS 100A 3-140-177 PROVISIONAL"
+		(property "Value" "UHS 100A 50V"
 			(at 274.32 67.31 90)
 			(show_name no)
@@
 			)
 		)
-		(property "Footprint" "PDB_Footprints:SCHURTER_UHS_8.4x9.4mm_PROVISIONAL"
+		(property "Footprint" "PDB_Footprints:Fuse_SCHURTER_UHS_8.4x9.4mm"
 			(at 274.32 74.168 90)
 			(hide yes)
@@
 			)
 		)
-		(property "Datasheet" "https://www.schurter.com/en/datasheet/UHS"
+		(property "Datasheet" "${KIPRJMOD}/Datasheets/SCHURTER_UHS.pdf"
 			(at 274.32 72.39 0)
 			(hide yes)
@@
 			)
 		)
-		(property "Description" "100 A surface-mount high-current fuse candidate for the dedicated ESC branch"
+		(property "Description" "Dedicated ESC branch: SCHURTER 3-140-177, 100 A, 50 VDC. This is overload backup; the ESC branch does not have active reverse-polarity protection."
 			(at 274.32 67.31 90)
 			(hide yes)
@@
 			)
 		)
-		(property "Selection_Status" "PROVISIONAL: verify 60 A continuous temperature rise, 100 A/30 s time-current behavior, 4S pack fault current, breaking capacity, and required heavy-copper land pattern."
+		(property "Selection_Status" "Selected prototype fuse. Manufacturer pad pattern 3.4 x 6.15 mm, 3.3 mm gap. 100 A/30 s target subject to ambient derating and assembly thermal test; pack fault duty must remain within breaking rating."
 			(at 274.32 72.39 0)
 			(hide yes)
@@
 	)
 	(symbol
-		(lib_id "Device:C")
+		(lib_id "PDB_Symbols:CP_Elec_Panasonic")
 		(at 322.58 78.74 0)
 		(unit 1)
@@
 			)
 		)
-		(property "Value" "470u 35V LOW-ESR"
+		(property "Value" "470u 35V HYBRID"
 			(at 326.39 80.01 0)
 			(show_name no)
@@
 			)
 		)
-		(property "Footprint" "Capacitor_SMD:CP_Elec_10x10.5"
+		(property "Footprint" "PDB_Footprints:CP_Elec_Panasonic_G16_10x16.5"
 			(at 323.5452 80.01 0)
 			(hide yes)
@@
 			)
 		)
-		(property "Datasheet" ""
+		(property "Datasheet" "${KIPRJMOD}/Datasheets/Panasonic_ZS.pdf"
 			(at 322.58 76.2 0)
 			(hide yes)
@@
 			)
 		)
-		(property "Description" "Local low-ESR bulk capacitor at ESC connector; final capacitance and ripple-current rating must be coordinated with the ESC vendor."
+		(property "Description" "Local supplemental ESC capacitor: 470 uF, 35 V, hybrid, 11 mOhm ESR at 100 kHz, 4 Arms at 100 kHz/125 C. Preserve the ESC manufacturer-required capacitor at the ESC."
 			(at 326.39 77.47 0)
 			(hide yes)
@@
 			)
 		)
-		(property "Selection_Status" "PROVISIONAL 4S value; use 35 V minimum rating and qualify ripple current, ESR, temperature, polarity, and inrush."
+		(property "Selection_Status" "Selected EEHZS1V471P G16; 10 mm diameter, 16.5 mm height. Additional ESC-side capacitor and harness transient/ripple tests required."
 			(at 322.58 76.2 0)
 			(hide yes)
@@
 			)
 		)
+		(property "MPN" "EEHZS1V471P"
+			(at 0 0 0)
+			(effects (font (size 1.27 1.27)) (hide yes))
+		)
+		(property "Manufacturer" "Panasonic"
+			(at 0 0 0)
+			(effects (font (size 1.27 1.27)) (hide yes))
+		)
 	)
 	(symbol
@@
 	)
 	(symbol
-		(lib_id "Connector_Generic:Conn_01x02")
+		(lib_id "PDB_Symbols:Conn_01x02_Phoenix")
 		(at 17.78 40.64 180)
 		(unit 1)
@@
 			)
 		)
-		(property "Value" "MKDSP 25/2-15.00 PROVISIONAL"
+		(property "Value" "MKDSP 25/2-15.00"
 			(at 17.78 35.56 0)
 			(show_name no)
@@
 			)
 		)
-		(property "Footprint" "PDB_Footprints:MKDSP25_2_15mm_PROVISIONAL"
+		(property "Footprint" "PDB_Footprints:Connector_MKDSP25_2_15mm"
 			(at 17.78 40.64 0)
 			(hide yes)
@@
 			)
 		)
-		(property "Selection_Status" "LAB DESIGN IN PROGRESS: verify exact terminal, footprint, conductor, wave-solder process, and power-path temperature before full-current use."
+		(property "Selection_Status" "Drawing checked 2026-10-01: 15 mm pole pitch, 3.8 mm paired pins, 12.5 mm row pitch, 1.6 mm holes. 125 A part rating is conditional on conductor and temperature; assembly and harness qualification required."
 			(at 17.78 40.64 0)
 			(hide yes)
@@
 			)
 		)
-		(property "Selection_Status" "PROVISIONAL: local transient suppressor only; not a substitute for ESC input capacitors or harness testing."
+		(property "Selection_Status" "SMBJ24CA retained for local ringing control. Clamp is not a 35 V ceiling; verify installed 4S harness waveforms and pulse energy."
 			(at 300.99 76.2 0)
 			(hide yes)
@@
 	)
 	(symbol
-		(lib_id "Connector_Generic:Conn_01x02")
+		(lib_id "PDB_Symbols:Conn_01x02_Phoenix")
 		(at 388.62 72.39 0)
 		(unit 1)
@@
 			)
 		)
-		(property "Value" "MKDSP 25/2-15.00 PROVISIONAL"
+		(property "Value" "MKDSP 25/2-15.00"
 			(at 388.62 67.31 0)
 			(show_name no)
@@
 			)
 		)
-		(property "Footprint" "PDB_Footprints:MKDSP25_2_15mm_PROVISIONAL"
+		(property "Footprint" "PDB_Footprints:Connector_MKDSP25_2_15mm"
 			(at 388.62 50.8 0)
 			(hide yes)
@@
 			)
 		)
-		(property "Selection_Status" "LAB DESIGN IN PROGRESS: verify exact terminal, footprint, conductor, wave-solder process, and power-path temperature before full-current use."
+		(property "Selection_Status" "Drawing checked 2026-10-01: 15 mm pole pitch, 3.8 mm paired pins, 12.5 mm row pitch, 1.6 mm holes. 125 A part rating is conditional on conductor and temperature; assembly and harness qualification required."
 			(at 388.62 50.8 0)
 			(hide yes)

Commit message: fixes 10.2.26
Parts:
- F1: value 4A MINI -> 7.5A MINI; MPN 0297004.WXNV -> 029707.5WXNV; Selection_Status 4 A 32 V MINI; load envelope 2.5 A maximum. Fuse, source an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 -> 7.5 A 32 V MINI selected for 5 A continuous avionics allowa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
- R5: Selection_Status 5 mOhm 1% 2 W four-terminal. Nominal breaker 10 A; normal-condition range 7.92-12.12 A. F1 remains 4 A; conductor/fuse coordination required. -> 5 mOhm 1% 2 W four-terminal. Nominal breaker 10 A; normal-condition range 7.92-12.12 A. F1 is 7.5 A for a 5 A continuous avionics allowance; conductor/fuse coordination required.
Changed lines of the file:
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@@
 			)
 		)
-		(property "Selection_Status" "5 mOhm 1% 2 W four-terminal. Nominal breaker 10 A; normal-condition range 7.92-12.12 A. F1 remains 4 A; conductor/fuse coordination required."
+		(property "Selection_Status" "5 mOhm 1% 2 W four-terminal. Nominal breaker 10 A; normal-condition range 7.92-12.12 A. F1 is 7.5 A for a 5 A continuous avionics allowance; conductor/fuse coordination required."
 			(at 187.96 -67.31 0)
 			(hide yes)
@@
 			)
 		)
-		(property "Value" "4A MINI"
+		(property "Value" "7.5A MINI"
 			(at 40.64 33.02 90)
 			(show_name no)
@@
 			)
 		)
-		(property "Description" "4 A, 32 VDC MINI blade fuse; backup protection for a fault the MOSFETs cannot interrupt"
+		(property "Description" "7.5 A, 32 VDC MINI blade fuse; backup protection for a fault the MOSFETs cannot interrupt"
 			(at 40.64 33.02 90)
 			(hide yes)
@@
 			)
 		)
-		(property "Selection_Status" "4 A 32 V MINI; load envelope 2.5 A maximum. Fuse, source and conductor coordination remains a release requirement."
+		(property "Selection_Status" "7.5 A 32 V MINI selected for 5 A continuous avionics allowance (67% of fuse rating). Electronic breaker remains nominally 10 A; fuse, source and conductor coordination remains a release requirement."
 			(at 40.64 38.1 0)
 			(hide yes)
@@
 			)
 		)
-		(property "MPN" "0297004.WXNV"
+		(property "MPN" "029707.5WXNV"
 			(at 40.64 38.1 0)
 			(hide yes)

Commit message: Prepare PDB Rev A JLCPCB prototype manufacturing package
Parts:
- C11, C12, C13, C14, C15, C16: footprint Capacitor_THT:C_Rect_L7.2mm_W4.5mm_P5.00mm -> PDB_Footprints:C_Rect_L7.2mm_W4.5mm_P5.00mm_JLC
- C18: MPN (none) -> C2012X7R1H105K125AB; Manufacturer (none) -> TDK; Selection_Status (none) -> Prototype selection: 1 uF 50 V X7R 10%, 0805. Nominal speci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
- C19: MPN (none) -> C0805C104K5RACTU; Manufacturer (none) -> KEMET; Selection_Status (none) -> Prototype selection: 100 nF 50 V X7R 10%, 0805. Nominal spe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
- D5: MPN (none) -> SMBJ24CA; Manufacturer (none) -> Bourns
- F1: Assembly_Note (none) -> Mount one Keystone 3568 holder at F1. Supply one Littelfuse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; Holder_Manufacturer Keystone Electronics -> Keystone
- J4: footprint Connector_AMASS:AMASS_XT60PW-F_1x02_P7.20mm_Horizontal -> PDB_Footprints:AMASS_XT60PW-F_1x02_P7.20mm_Horizontal
Changed lines of the file:
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@@
 		(in_pos_files yes)
 		(dnp no)
+		(property "MPN" "C2012X7R1H105K125AB"
+			(at 345.44 78.74 0)
+			(hide yes)
+			(effects (font (size 1 1)))
+		)
+		(property "Manufacturer" "TDK"
+			(at 345.44 78.74 0)
+			(hide yes)
+			(effects (font (size 1 1)))
+		)
+		(property "Selection_Status" "Prototype selection: 1 uF 50 V X7R 10%, 0805. Nominal specifications verified against manufacturer; installed bias/ripple validation pending."
+			(at 345.44 78.74 0)
+			(hide yes)
+			(effects (font (size 1 1)))
+		)
 		(property "Reference" "C18"
 			(at 349.25 77.47 0)
@@
 			)
 		)
-		(property "Datasheet" ""
+		(property "Datasheet" "https://product.tdk.com/en/search/capacitor/ceramic/mlcc/info?part_no=C2012X7R1H105K125AB"
 			(at 345.44 76.2 0)
 			(hide yes)
@@
 			)
 		)
-		(property "Footprint" "Capacitor_THT:C_Rect_L7.2mm_W4.5mm_P5.00mm"
+		(property "Footprint" "PDB_Footprints:C_Rect_L7.2mm_W4.5mm_P5.00mm_JLC"
 			(at 355.6 241.3 0)
 			(hide yes)
@@
 			)
 		)
-		(property "Footprint" "Capacitor_THT:C_Rect_L7.2mm_W4.5mm_P5.00mm"
+		(property "Footprint" "PDB_Footprints:C_Rect_L7.2mm_W4.5mm_P5.00mm_JLC"
 			(at 140.97 91.44 0)
 			(hide yes)
@@
 			)
 		)
-		(property "Footprint" "Capacitor_THT:C_Rect_L7.2mm_W4.5mm_P5.00mm"
+		(property "Footprint" "PDB_Footprints:C_Rect_L7.2mm_W4.5mm_P5.00mm_JLC"
 			(at 322.58 162.56 0)
 			(hide yes)
@@
 			)
 		)
-		(property "Footprint" "Connector_AMASS:AMASS_XT60PW-F_1x02_P7.20mm_Horizontal"
+		(property "Footprint" "PDB_Footprints:AMASS_XT60PW-F_1x02_P7.20mm_Horizontal"
 			(at 388.62 35.56 0)
 			(hide yes)
@@
 			)
 		)
-		(property "Footprint" "Capacitor_THT:C_Rect_L7.2mm_W4.5mm_P5.00mm"
+		(property "Footprint" "PDB_Footprints:C_Rect_L7.2mm_W4.5mm_P5.00mm_JLC"
 			(at 30.48 104.14 0)
 			(hide yes)
@@
 			)
 		)
-		(property "Footprint" "Capacitor_THT:C_Rect_L7.2mm_W4.5mm_P5.00mm"
+		(property "Footprint" "PDB_Footprints:C_Rect_L7.2mm_W4.5mm_P5.00mm_JLC"
 			(at 129.54 91.44 0)
 			(hide yes)
@@
 		(dnp no)
 		(fields_autoplaced yes)
+		(property "Assembly_Note" "Mount one Keystone 3568 holder at F1. Supply one Littelfuse 029707.5WXNV separately and insert after soldering. Do not treat blade fuse as an SMT placement."
+			(at 40.64 38.1 0)
+			(hide yes)
+			(effects (font (size 1 1)))
+		)
 		(property "Reference" "F1"
 			(at 40.64 30.48 90)
@@
 			)
 		)
-		(property "Holder_Manufacturer" "Keystone Electronics"
+		(property "Holder_Manufacturer" "Keystone"
 			(at 40.64 38.1 0)
 			(hide yes)
@@
 			)
 		)
-		(property "Footprint" "Capacitor_THT:C_Rect_L7.2mm_W4.5mm_P5.00mm"
+		(property "Footprint" "PDB_Footprints:C_Rect_L7.2mm_W4.5mm_P5.00mm_JLC"
 			(at 347.98 208.28 0)
 			(hide yes)
@@
 		(in_pos_files yes)
 		(dnp no)
+		(property "MPN" "SMBJ24CA"
+			(at 300.99 78.74 0)
+			(hide yes)
+			(effects (font (size 1 1)))
+		)
+		(property "Manufacturer" "Bourns"
+			(at 300.99 78.74 0)
+			(hide yes)
+			(effects (font (size 1 1)))
+		)
 		(property "Reference" "D5"
 			(at 304.8 77.47 90)
@@
 			)
 		)
-		(property "Datasheet" ""
+		(property "Datasheet" "https://www.bourns.com/docs/product-datasheets/smbj.pdf"
 			(at 300.99 76.2 0)
 			(hide yes)
@@
 		(in_pos_files yes)
 		(dnp no)
+		(property "MPN" "C0805C104K5RACTU"
+			(at 363.22 78.74 0)
+			(hide yes)
+			(effects (font (size 1 1)))
+		)
+		(property "Manufacturer" "KEMET"
+			(at 363.22 78.74 0)
+			(hide yes)
+			(effects (font (size 1 1)))
+		)
+		(property "Selection_Status" "Prototype selection: 100 nF 50 V X7R 10%, 0805. Nominal specifications verified against manufacturer; installed transient validation pending."
+			(at 363.22 78.74 0)
+			(hide yes)
+			(effects (font (size 1 1)))
+		)
 		(property "Reference" "C19"
 			(at 367.03 77.47 0)
@@
 			)
 		)
-		(property "Datasheet" ""
+		(property "Datasheet" "https://search.kemet.com/download/specsheet/C0805C104K5RACTU"
 			(at 363.22 76.2 0)
 			(hide yes)
