File: Osiris_PDB_RevA.kicad_pcb (KiCad board)
At the start: 2 copper layers, 291.2 x 129.8 mm, 47 parts, among them J1 XT60PW-M, J2 OSIRIS_I2C, J3 XT60PW-F, Q1 ISC015N06NM5LF2, Q2 ISC015N06NM5LF2, U1 LTC4368IMS-1-PBF, U2 INA228AIDGSR, U3 LT3010EMS8E, U4 74AUP1G07GW

Commit message: 9/18.2026
Parts:
- added C11: 1u, Capacitor_THT:C_Rect_L7.2mm_W4.5mm_P5.00mm, F.Cu at (74.5, 40.0)
- added C12: 1u, Capacitor_THT:C_Rect_L7.2mm_W4.5mm_P5.00mm, F.Cu at (-22.6, 28.1)
- added C13: 1u, Capacitor_THT:C_Rect_L7.2mm_W4.5mm_P5.00mm, F.Cu at (-22.6, 34.1)
- added C14: 1u, Capacitor_THT:C_Rect_L7.2mm_W4.5mm_P5.00mm, F.Cu at (-22.6, 40.2)
- added C15: 1u, Capacitor_THT:C_Rect_L7.2mm_W4.5mm_P5.00mm, F.Cu at (-22.6, 46.2)
- added C16: 1u, Capacitor_THT:C_Rect_L7.2mm_W4.5mm_P5.00mm, F.Cu at (53.5, 49.0)
- added D4: SMAJ24CA, Diode_SMD:D_SMA, F.Cu at (65.0, 38.0)
- added Q3: BSC070N10NS5, Package_TO_SOT_SMD:TDSON-8-1, F.Cu at (69.7, 29.6)
- added R19: 1k, Resistor_SMD:R_2512_6332Metric, F.Cu at (53.0, 40.0)
- added R20: 1, Resistor_SMD:R_2512_6332Metric, F.Cu at (58.0, 46.0)
- added R21: 100, Resistor_SMD:R_0805_2012Metric, F.Cu at (-13.5, 46.2)
- added U5: LTC4359IMS8, Package_SO:MSOP-8_3x3mm_P0.65mm, F.Cu at (65.0, 45.0)
- D3: value MBR0540 -> STPST10H100SB; footprint Diode_SMD:D_SOD-123 -> PDB_Footprints:STPST10H100SB_DPAK
- moved R11 76.8 mm to (157.2, 70.8), turned to 180 degrees
- moved D3 76.1 mm to (141.0, 27.4), turned to -90 degrees
- moved U2 70.5 mm to (149.2, 34.5), turned to 90 degrees
- moved C4 70.2 mm to (145.0, 23.7), turned to -90 degrees
- moved Q1 67.8 mm to (84.1, 29.9)
- moved Q2 65.1 mm to (92.0, 29.9), turned to 180 degrees
- moved C10 63.7 mm to (164.0, 70.8), turned to 180 degrees
- moved U3 61.6 mm to (149.4, 26.3), turned to 180 degrees
- moved R2 60.9 mm to (45.9, 74.2)
- moved C1 60.9 mm to (57.9, 66.5)
- moved C2 60.9 mm to (58.6, 74.7)
- moved R1 60.9 mm to (41.6, 74.2)
- moved R13 60.9 mm to (45.9, 77.7)
- moved R4 60.9 mm to (57.9, 70.5)
- moved R5 60.9 mm to (63.5, 69.7)
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Connections:
- F1 pad 2: /VBAT_FUSED -> /IDEAL_IN
- TP1 pad 1: /VBAT_FUSED -> /IDEAL_IN
- U2 pad 8: /PDB_VOUT -> /INA_VBUS
Routing:
- added copper zone on F.Cu, net GND

Commit message: routing main power path 25%
Parts:
- U1: value LTC4368IMS-1-PBF -> LTC4368HMS-1-PBF
- moved R5 123.9 mm to (142.6, -25.6)
- moved R15 107.6 mm to (49.5, 14.2)
- moved U2 92.7 mm to (125.0, 123.9), turned to 0 degrees
- moved C15 92.5 mm to (69.0, 33.5), turned to -90 degrees
- moved U3 90.1 mm to (124.9, 113.0)
- moved C1 76.8 mm to (67.7, -9.66)
- moved C2 76.8 mm to (68.4, -1.46)
- moved R4 76.8 mm to (67.7, -5.71)
- moved C3 72.6 mm to (63.2, 11.0), turned to 90 degrees
- moved Q2 70.0 mm to (134.6, -25.6), turned to 0 degrees
- moved R13 66.8 mm to (67.5, 14.5)
- moved R6 65.7 mm to (59.4, 11.9), turned to 90 degrees
- moved R7 65.6 mm to (57.4, 11.9), turned to -90 degrees
- moved R14 62.9 mm to (118.4, 95.0)
- moved TP2 62.9 mm to (123.9, 82.5)
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Routing:
- net /IDEAL_GATE: track 0.00 -> 2.95 mm
- added copper zone on F.Cu, net /IDEAL_IN
- added copper zone on F.Cu, net /INPUT_DAMP
- added copper zone on F.Cu, net /VBAT_RAW

Commit message: Save current PDB schematic and layout updates
Parts:
- added H1: MountingHole, MountingHole:MountingHole_3.2mm_M3_ISO14580, F.Cu at (45.5, 18.8)
- added H2: MountingHole, MountingHole:MountingHole_3.2mm_M3_ISO14580, F.Cu at (90.5, 18.8)
- added H3: MountingHole, MountingHole:MountingHole_3.2mm_M3_ISO14580, F.Cu at (90.5, 58.8)
- added H4: MountingHole, MountingHole:MountingHole_3.2mm_M3_ISO14580, F.Cu at (45.5, 58.8)
- added J4: XT60PW-F, Connector_AMASS:AMASS_XT60PW-F_1x02_P7.20mm_Horizontal, F.Cu at (92.1, 51.5)
- R17, R18: moved to B.Cu
- moved J2 183.7 mm to (81.2, 51.6), turned to 180 degrees
- moved J3 171.3 mm to (92.2, 34.8)
- moved R12 168.8 mm to (75.8, 45.5)
- moved C7 162.8 mm to (60.0, 43.5), turned to 90 degrees
- moved R8 157.5 mm to (71.5, 23.8), turned to 180 degrees
- moved C8 144.9 mm to (46.8, 44.0), turned to 90 degrees
- moved R9 140.3 mm to (76.2, 35.0), turned to -90 degrees
- moved TP3 136.2 mm to (78.5, 14.8)
- moved TP4 132.4 mm to (82.0, 14.8)
- moved TP5 131.7 mm to (50.0, 53.2)
- moved R16 129.8 mm to (52.0, 45.5)
- moved C5 125.4 mm to (56.5, 41.8), turned to 180 degrees
- moved TP7 119.8 mm to (57.2, 53.2)
- moved TP6 114.0 mm to (53.8, 53.2)
- moved U4 109.7 mm to (55.8, 45.8), turned to 90 degrees
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Routing:
- net /PDB_VOUT: track 0.00 -> 92.4 mm, vias 0 -> 6
- net /PDB_3V3: track 0.00 -> 67.6 mm, vias 0 -> 3
- net /PDB_FAULT_N: track 0.00 -> 43.5 mm, vias 0 -> 3
- net /SHUNT_HI: track 0.00 -> 37.5 mm, vias 0 -> 5
- net /GATE_PIN: track 0.00 -> 36.9 mm, vias 0 -> 4
- net /INA_IN_N: track 0.00 -> 34.5 mm, vias 0 -> 2
- net /INA_VBUS: track 0.00 -> 32.6 mm
- net /SHUNT_LO: track 0.00 -> 32.5 mm, vias 0 -> 2
- net /PDB_I2C_SCL: track 0.00 -> 25.1 mm, vias 0 -> 4
- net /PDB_I2C_SDA: track 0.00 -> 22.8 mm, vias 0 -> 4
- net /LTC_UV: track 0.00 -> 22.3 mm
- net /INA_IN_P: track 0.00 -> 20.9 mm, vias 0 -> 1
- net /INA_ALERT_LOCAL_N: track 0.00 -> 20.8 mm, vias 0 -> 2
- net /IDEAL_VSS: track 0.00 -> 20.7 mm
- net /VBAT_FUSED: track 0.00 -> 19.3 mm, vias 0 -> 5
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- added copper zone on F.Cu, net /INA_IN_P
- added copper zone on B.Cu, net /PDB_PROTECTED
- added copper zone on F.Cu, net /PDB_PROTECTED
- added copper zone on B.Cu, net /PDB_VOUT
- added copper zone on F.Cu, net /PDB_VOUT
- added copper zone on F.Cu, net /SW_COMMON
- added copper zone on B.Cu, net /VBAT_FUSED
- added copper zone on F.Cu, net /VBAT_FUSED
- added copper zone on B.Cu, net GND
Other:
- board size 291.2 x 129.8 mm -> 94.5 x 51.8 mm
- board text added: "BATT IN"
- board text added: "GND"
- board text added: "IDEAL IN"
- board text added: "INA ALERT"
- board text added: "OUT"
- board text added: "PDB 3V3"
- board text added: "PDB FAULT"
- board text added: "PDB_PROT"
- board text added: "PDB_VOUT"
