File: Osiris_PDB_RevA.kicad_pcb (KiCad board)
At the start: 4 copper layers, 127.5 x 65 mm, 69 parts, among them J1 MKDSP 25/2-15.00, J2 OSIRIS_I2C, J3 MKDSP 25/2-15.00, J4 XT60PW-F, Q1 ISC015N06NM5LF2, Q2 ISC015N06NM5LF2, Q3 BSC070N10NS5, U1 LTC4368HMS-1-PBF, U2 INA228AIDGSR, U3 LT3010EMS8E, U4 74AUP1G07GW, U5 LTC4359IMS8

Commit message: Update REV1.1 XT60 PDB and publish clean JLCPCB outputs
Parts:
- C17: value 470u 35V HYBRID -> 330u 50V HYBRID
- D5: value SMBJ24CA -> SMBJ18CA
- J1, J3: value MKDSP 25/2-15.00 -> XT60PW-F; footprint PDB_Footprints:Connector_MKDSP25_2_15mm -> PDB_Footprints:AMASS_XT60PW-F_1x02_P7.20mm_Horizontal_EdgeMounted
- J4: footprint PDB_Footprints:AMASS_XT60PW-F_1x02_P7.20mm_Horizontal -> PDB_Footprints:AMASS_XT60PW-F_1x02_P7.20mm_Horizontal_EdgeMounted
- moved J1 16.1 mm to (119.0, 92.0), turned to 90 degrees
- moved J3 15.2 mm to (184.0, 93.0), turned to -90 degrees
Routing:
- net GND: vias 157 -> 151
Other:
- board size 127.5 x 65 mm -> 82.5 x 65 mm
- board text added: "XT60 LC 1/0.5oz"
- board text removed: "LC TEST 1/0.5oz"

Commit message: Update INA238 telemetry, ESC capacitor bank and procurement outputs
Parts:
- added C20: 220u 50V HYBRID, PDB_Footprints:CP_Elec_Panasonic_G16_10x16.5_ZS, F.Cu at (172.3, 74.8)
- C17: value 330u 50V HYBRID -> 220u 50V HYBRID; footprint PDB_Footprints:CP_Elec_Panasonic_G16_10x16.5 -> PDB_Footprints:CP_Elec_Panasonic_G16_10x16.5_ZS
- U2: value INA228AIDGSR -> INA238AIDGSR
Routing:
- net GND: track 20.3 -> 32.3 mm, vias 151 -> 157
